File: hardware/CH592/OpenController-CH592.kicad_sch (KiCad schematic)
At the start: 10 parts, among them J1 Castellated, U1 CH592D, U2 XC6206P332MR-G, Y1 32MHz

Commit message: hardware: keep the CH592 exposed-pad paste off its thermal vias
The same fix as for the CH572: the exposed pad's four GND vias sat inside
the paste windows, so solder could wick into the open barrels during
reflow (CodeRabbit review on #34).

U1's CH592D footprint now has four 0.4/0.2 mm thermal vias built in,
0.7 mm from the centre along each axis, and its paste is a central
window plus four edge windows covering about 53% of the 1.9 mm pad, each
at least 0.075 mm clear of the via copper. The separate board vias in
the pad are gone, and the bottom-layer SWDIO run now crosses under U1
between the two rows of thermal vias. ERC and DRC (with schematic
parity) report no violations.

Co-Authored-By: Claude Opus 5.5 <noreply@anthropic.com>
Parts:
- U1: footprint OpenController:QFN-20-1EP_3x3mm_P0.4mm_EP1.9x1.9mm -> OpenController:QFN-20-1EP_3x3mm_P0.4mm_EP1.9x1.9mm_ThermalVias
Changed lines of the file:
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@@
 			)
 		)
-		(property "Footprint" "OpenController:QFN-20-1EP_3x3mm_P0.4mm_EP1.9x1.9mm"
+		(property "Footprint" "OpenController:QFN-20-1EP_3x3mm_P0.4mm_EP1.9x1.9mm_ThermalVias"
 			(at 148.59 72.39 0)
 			(hide yes)

Commit message: hardware: draw the CH592D QFN footprint for OpenController
U1's footprint started from a copy of KiCad's QFN-20 footprint, which
KiCad's CC-BY-SA 4.0 library licence does not let a CERN-OHL-W project
library carry as a separate file (Codex review). It is now drawn from
scratch from the CH592 datasheet's QFN20 drawing, with the same
geometry as before:
- lands 1.20 to 1.85 mm from the centre;
- a 1.9 mm exposed-pad land with four 0.4/0.2 mm tented thermal vias at
  (+/-0.7, +/-0.7) mm;
- the same paste windows.
hardware/NOTICE records its provenance alongside the CH572D footprint.

README corrections from the same review: paste coverage is 51% once the
windows' rounded corners are counted (not 53%); the closest plated pad
holes are the thermal vias, 1.2 mm apart; and the lead overhang at a
land's inner end is 0.02 mm on a nominal body but up to 0.07 mm on the
smallest 2.9 mm body. ERC and DRC (with schematic parity) report no
violations.

Co-Authored-By: Claude Opus 5.5 <noreply@anthropic.com>
Parts:
- U1: footprint OpenController:QFN-20-1EP_3x3mm_P0.4mm_EP1.9x1.9mm_ThermalVias -> OpenController:CH592D_QFN-20_3x3mm_P0.4mm_EP1.9mm_ThermalVias
Changed lines of the file:
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@@
 			)
 		)
-		(property "Footprint" "OpenController:QFN-20-1EP_3x3mm_P0.4mm_EP1.9x1.9mm_ThermalVias"
+		(property "Footprint" "OpenController:CH592D_QFN-20_3x3mm_P0.4mm_EP1.9mm_ThermalVias"
 			(at 148.59 72.39 0)
 			(hide yes)
